File: Version 2/main.sch (EAGLE design)
At the start: 28 parts, among them IC1 LM324N, IC2 LM339N, Q1 BC487, Q2 BC487, Q3 BC487, Q4 BC487

Commit message: Finished 2nd Version
Parts:
- R15, R16, R17, R18: value 68Ω -> IR
Changed lines of the file:
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@@
 <part name="R14" library="resistor" deviceset="R-US_" device="0204/7" value="3kΩ"/>
 <part name="SUPPLY5" library="supply2" deviceset="GND" device=""/>
-<part name="R15" library="resistor" deviceset="R-US_" device="0204/7" value="68Ω"/>
-<part name="R16" library="resistor" deviceset="R-US_" device="0204/7" value="68Ω"/>
-<part name="R17" library="resistor" deviceset="R-US_" device="0204/7" value="68Ω"/>
-<part name="R18" library="resistor" deviceset="R-US_" device="0204/7" value="68Ω"/>
+<part name="R15" library="resistor" deviceset="R-US_" device="0204/7" value="IR"/>
+<part name="R16" library="resistor" deviceset="R-US_" device="0204/7" value="IR"/>
+<part name="R17" library="resistor" deviceset="R-US_" device="0204/7" value="IR"/>
+<part name="R18" library="resistor" deviceset="R-US_" device="0204/7" value="IR"/>
 <part name="SUPPLY6" library="supply2" deviceset="GND" device=""/>
 </parts>
@@
 <wire x1="-48.26" y1="93.98" x2="-40.64" y2="93.98" width="0.1524" layer="91"/>
 <label x="-40.64" y="93.98" size="1.778" layer="95" xref="yes"/>
+<junction x="-48.26" y="86.36"/>
 </segment>
 </net>
@@
 </segment>
 <segment>
-<pinref part="R3" gate="G$1" pin="2"/>
-<wire x1="17.78" y1="5.08" x2="25.4" y2="5.08" width="0.1524" layer="91"/>
 <wire x1="25.4" y1="5.08" x2="25.4" y2="12.7" width="0.1524" layer="91"/>
 <pinref part="IC1" gate="C" pin="OUT"/>
@@
 <wire x1="25.4" y1="12.7" x2="55.88" y2="12.7" width="0.1524" layer="91"/>
 <junction x="25.4" y="12.7"/>
+<pinref part="R3" gate="G$1" pin="2"/>
+<wire x1="25.4" y1="5.08" x2="17.78" y2="5.08" width="0.1524" layer="91"/>
 </segment>
 <segment>
@@
 </sheet>
 </sheets>
+<errors>
+</errors>
 </schematic>
 </drawing>

Commit message: Final Version
Parts:
- R1, R2, R3, R4: value TRA -> 68kΩ
- R10, R11, R12, R13, R14, R9: value 3kΩ -> 3k3Ω
- R15, R16, R17, R18: value IR -> 44Ω
- R5, R6, R7, R8: value 68Ω -> 100Ω
Connections:
- net IRVCC renamed +1.84V
Changed lines of the file:
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@@
 <setting verticaltext="up"/>
 </settings>
-<grid distance="0.1" unitdist="inch" unit="inch" style="lines" multiple="1" display="yes" altdistance="0.01" altunitdist="inch" altunit="inch"/>
+<grid distance="0.1" unitdist="inch" unit="inch" style="lines" multiple="1" display="no" altdistance="0.01" altunitdist="inch" altunit="inch"/>
 <layers>
 <layer number="1" name="Top" color="4" fill="1" visible="no" active="no"/>
@@
 <parts>
 <part name="IC1" library="linear" deviceset="LM324" device="N"/>
-<part name="R1" library="resistor" deviceset="R-US_" device="0204/7" value="TRA"/>
+<part name="R1" library="resistor" deviceset="R-US_" device="0204/7" value="68kΩ"/>
 <part name="SV1" library="con-lstb" deviceset="MA08-1" device="" value="Photodiode Connectors"/>
 <part name="SV2" library="con-lstb" deviceset="MA08-1" device="" value="IR LED Connectors"/>
 <part name="SV3" library="con-lstb" deviceset="MA08-1" device="" value="Visual LED Connector"/>
-<part name="R2" library="resistor" deviceset="R-US_" device="0204/7" value="TRA"/>
-<part name="R3" library="resistor" deviceset="R-US_" device="0204/7" value="TRA"/>
-<part name="R4" library="resistor" deviceset="R-US_" device="0204/7" value="TRA"/>
+<part name="R2" library="resistor" deviceset="R-US_" device="0204/7" value="68kΩ"/>
+<part name="R3" library="resistor" deviceset="R-US_" device="0204/7" value="68kΩ"/>
+<part name="R4" library="resistor" deviceset="R-US_" device="0204/7" value="68kΩ"/>
 <part name="SUPPLY1" library="supply2" deviceset="GND" device=""/>
 <part name="IC2" library="linear" deviceset="LM339" device="N"/>
@@
 <part name="Q3" library="transistor-npn" deviceset="BC487*" device=""/>
 <part name="Q4" library="transistor-npn" deviceset="BC487*" device=""/>
-<part name="R5" library="resistor" deviceset="R-US_" device="0204/7" value="68Ω"/>
-<part name="R6" library="resistor" deviceset="R-US_" device="0204/7" value="68Ω"/>
-<part name="R7" library="resistor" deviceset="R-US_" device="0204/7" value="68Ω"/>
-<part name="R8" library="resistor" deviceset="R-US_" device="0204/7" value="68Ω"/>
-<part name="R9" library="resistor" deviceset="R-US_" device="0204/7" value="3kΩ"/>
-<part name="R10" library="resistor" deviceset="R-US_" device="0204/7" value="3kΩ"/>
-<part name="R11" library="resistor" deviceset="R-US_" device="0204/7" value="3kΩ"/>
-<part name="R12" library="resistor" deviceset="R-US_" device="0204/7" value="3kΩ"/>
+<part name="R5" library="resistor" deviceset="R-US_" device="0204/7" value="100Ω"/>
+<part name="R6" library="resistor" deviceset="R-US_" device="0204/7" value="100Ω"/>
+<part name="R7" library="resistor" deviceset="R-US_" device="0204/7" value="100Ω"/>
+<part name="R8" library="resistor" deviceset="R-US_" device="0204/7" value="100Ω"/>
+<part name="R9" library="resistor" deviceset="R-US_" device="0204/7" value="3k3Ω"/>
+<part name="R10" library="resistor" deviceset="R-US_" device="0204/7" value="3k3Ω"/>
+<part name="R11" library="resistor" deviceset="R-US_" device="0204/7" value="3k3Ω"/>
+<part name="R12" library="resistor" deviceset="R-US_" device="0204/7" value="3k3Ω"/>
 <part name="SUPPLY3" library="supply2" deviceset="GND" device=""/>
 <part name="SV4" library="con-lstb" deviceset="MA04-1" device="" value="Power In"/>
 <part name="SUPPLY4" library="supply2" deviceset="GND" device=""/>
-<part name="R13" library="resistor" deviceset="R-US_" device="0204/7" value="3kΩ"/>
-<part name="R14" library="resistor" deviceset="R-US_" device="0204/7" value="3kΩ"/>
+<part name="R13" library="resistor" deviceset="R-US_" device="0204/7" value="3k3Ω"/>
+<part name="R14" library="resistor" deviceset="R-US_" device="0204/7" value="3k3Ω"/>
 <part name="SUPPLY5" library="supply2" deviceset="GND" device=""/>
-<part name="R15" library="resistor" deviceset="R-US_" device="0204/7" value="IR"/>
-<part name="R16" library="resistor" deviceset="R-US_" device="0204/7" value="IR"/>
-<part name="R17" library="resistor" deviceset="R-US_" device="0204/7" value="IR"/>
-<part name="R18" library="resistor" deviceset="R-US_" device="0204/7" value="IR"/>
+<part name="R15" library="resistor" deviceset="R-US_" device="0204/7" value="44Ω"/>
+<part name="R16" library="resistor" deviceset="R-US_" device="0204/7" value="44Ω"/>
+<part name="R17" library="resistor" deviceset="R-US_" device="0204/7" value="44Ω"/>
+<part name="R18" library="resistor" deviceset="R-US_" device="0204/7" value="44Ω"/>
 <part name="SUPPLY6" library="supply2" deviceset="GND" device=""/>
 </parts>
@@
 </segment>
 </net>
-<net name="IRVCC" class="0">
+<net name="+1.84V" class="0">
 <segment>
 <pinref part="SV2" gate="1" pin="5"/>
