File: Version 2/main.brd (EAGLE design)
At the start: 42.9 x 49.5 mm, 28 parts, among them IC1 LM324N, IC2 LM339N, Q1 BC487, Q2 BC487, Q3 BC487, Q4 BC487

Commit message: 3-23-17 Periodic Push
Connections:
- net N$10 renamed T2
- net N$11 renamed T1
- net N$2 renamed AS1
- net N$3 renamed AS2
- net N$7 renamed AS4
- net N$8 renamed T3
- net N$9 renamed T4
- new net AS3: IC1.8, IC2.8, R3.2
- net VLOGIC: no longer IC1.8, IC2.8, R3.2
Routing:
- net PD1: track 94.7 -> 40.9 mm, vias 1 -> 0
- net VLOGIC: track 103.6 -> 55.8 mm
- net AS3: track 0.00 -> 45.5 mm
- net PD3: track 82.0 -> 105.5 mm, vias 0 -> 2
- net T2: track 89.4 -> 69.0 mm, vias 1 -> 3
- net AS2: track 57.2 -> 37.0 mm, vias 1 -> 3
- net T1: track 61.1 -> 75.9 mm
- net N$5: track 41.4 -> 27.9 mm
- net N$1: track 50.0 -> 63.3 mm, vias 0 -> 2
- net N$4: track 45.7 -> 33.6 mm, vias 2 -> 3
- net GND: track 112.2 -> 124.3 mm
- net PD2: track 59.5 -> 70.8 mm, vias 2 -> 0
- net T3: track 55.0 -> 44.6 mm
- net 5V: track 117.3 -> 124.1 mm
- net AS4: track 48.9 -> 42.7 mm, vias 1 -> 2
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